File: pcb/card34.kicad_pcb (KiCad board)
At the start: 2 copper layers, 208.8 x 20 mm, 77 parts, among them SW10 SW_PUSH, SW11 SW_PUSH, SW12 SW_PUSH, SW14 SW_PUSH, SW15 SW_PUSH, SW16 SW_PUSH, SW16 SW_Push, SW17 SW_PUSH, SW18 SW_PUSH, SW19 SW_PUSH, SW2 SW_PUSH, SW20 SW_PUSH, SW21 SW_PUSH, SW23 SW_PUSH, SW24 SW_PUSH, SW25 SW_PUSH, SW26 SW_PUSH, SW27 SW_PUSH, SW29 SW_PUSH, SW3 SW_PUSH, SW30 SW_PUSH, SW31 SW_PUSH, SW32 SW_PUSH, SW33 SW_PUSH, SW35 SW_PUSH, SW36 SW_PUSH, SW37 SW_PUSH, SW38 SW_PUSH, SW39 SW_PUSH, SW4 SW_PUSH, SW40 SW_PUSH, SW41 SW_PUSH, SW42 SW_PUSH, SW5 SW_PUSH, SW6 SW_PUSH, SW8 SW_PUSH, SW9 SW_PUSH, U1 ProMicro, U2 ProMicro

Commit message: folders rearranged
Parts:
- removed D10, D11, D12, D14, D15, D16, D17, D18, D19, D2, D20, D21, D23, D24, D25, D26, D27, D29, D3, D30, D31, D32, D33, D35, D36, D37, D38, D39, D4, D40, D41, D42, D5, D6, D8, D9: D, kbd:D3_TH_SMD_v2
- removed RSW2: SW_PUSH, kbd:ResetSW_1side
- removed the SW16 at (108.1, 76.8)
- removed the SW16 at (161.3, 150.6)
- removed SW19, SW23, SW24, SW25, SW26, SW27, SW29, SW30, SW31, SW32, SW33, SW35, SW36, SW37, SW38, SW39, SW40, SW41, SW42: SW_PUSH, kbd:keyswitch_cherrymx_alps_choc12_1u
- removed the SW2 at (70.1, 38.8)
- removed U2: ProMicro, kbd:ProMicro_v3
- added ?: , , F.Cu at (49.0, 43.5)
- added ?: , , F.Cu at (103.0, 77.5)
- added ?: , , F.Cu at (103.0, 43.5)
- added ?: , , F.Cu at (43.8, 89.9)
- added B+: MountingHole_Pad, kbd:1pin_conn, F.Cu at (34.9, 79.3)
- added B-: MountingHole_Pad, kbd:1pin_conn, F.Cu at (34.9, 94.5)
- added POWER SW: SW_SPDT, Kailh:SPDT_C128955, B.Cu at (35.2, 87.4)
- added SW16: SW_Push, Kailh:SW_PG1350_rev_DPB, F.Cu at (76.0, 69.0)
- added SW2: SW_Push, Kailh:SW_PG1350_rev_DPB, F.Cu at (40.0, 35.0)
- added SW2: SW_SPDT, Kailh:SPDT_C128955r, F.Cu at (35.2, 87.4)
- RSW1: value SW_PUSH -> SW_Push; footprint kbd:ResetSW_1side -> kbd:ResetSW
- SW10, SW11, SW12, SW14, SW15, SW17, SW18, SW20, SW21, SW3, SW4, SW5, SW6, SW8, SW9: value SW_PUSH -> SW_Push; footprint kbd:keyswitch_cherrymx_alps_choc12_1u -> Kailh:SW_PG1350_rev_DPB
- U1: value ProMicro -> ProMicro-kbd; footprint kbd:ProMicro_v3 -> kbd:ProMicro_v2
- moved SW21 53.0 mm to (94.0, 86.0)
- moved SW18 34.9 mm to (112.0, 69.0)
- moved SW12 34.6 mm to (112.0, 52.0)
- moved SW6 34.3 mm to (112.0, 35.0)
- moved SW17 34.0 mm to (94.0, 69.0)
- moved SW11 33.6 mm to (94.0, 52.0)
- moved SW5 33.3 mm to (94.0, 35.0)
- moved SW10 32.6 mm to (76.0, 52.0)
- moved SW4 32.3 mm to (76.0, 35.0)
- moved SW15 32.0 mm to (58.0, 69.0)
- moved SW9 31.6 mm to (58.0, 52.0)
- moved SW3 31.3 mm to (58.0, 35.0)
- moved SW14 31.1 mm to (40.0, 69.0)
- moved SW8 30.6 mm to (40.0, 52.0)
- moved U1 27.0 mm to (51.9, 86.9)
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Connections:
- net VCC renamed vcc
- net data renamed Switch18
- RSW1 pad 1: reset -> gnd
- RSW1 pad 2: GND -> reset
- SW10 pad 1: col3 -> Switch8
- SW10 pad 2: Net-(D10-Pad2) -> gnd
- SW11 pad 1: col4 -> Switch9
- SW11 pad 2: Net-(D11-Pad2) -> gnd
- SW12 pad 1: col5 -> Switch10
- SW12 pad 2: Net-(D12-Pad2) -> gnd
- SW14 pad 1: col1 -> Switch11
- SW14 pad 2: Net-(D14-Pad2) -> gnd
- SW15 pad 1: col2 -> Switch12
- SW15 pad 2: Net-(D15-Pad2) -> gnd
- SW17 pad 1: col4 -> Switch14
- SW17 pad 2: Net-(D17-Pad2) -> gnd
- SW18 pad 1: col5 -> Switch15
- SW18 pad 2: Net-(D18-Pad2) -> gnd
- SW20 pad 1: col4 -> Switch17
- SW20 pad 2: Net-(D20-Pad2) -> gnd
- SW21 pad 1: col5 -> Switch16
- SW21 pad 2: Net-(D21-Pad2) -> gnd
- SW3 pad 1: col2 -> Switch2
- SW3 pad 2: Net-(D3-Pad2) -> gnd
- SW4 pad 1: col3 -> Switch3
- SW4 pad 2: Net-(D4-Pad2) -> gnd
- SW5 pad 1: col4 -> Switch4
- SW5 pad 2: Net-(D5-Pad2) -> gnd
- SW6 pad 1: col5 -> Switch5
- SW6 pad 2: Net-(D6-Pad2) -> gnd
- SW8 pad 1: col1 -> Switch6
- SW8 pad 2: Net-(D8-Pad2) -> gnd
- SW9 pad 1: col2 -> Switch7
- SW9 pad 2: Net-(D9-Pad2) -> gnd
- U1 pad 1: Net-(U1-Pad1) -> Switch10
- U1 pad 10: row3 -> Switch1
- U1 pad 11: Net-(U1-Pad11) -> Switch16
- U1 pad 12: Net-(U1-Pad12) -> Switch17
- U1 pad 13: Net-(U1-Pad13) -> Switch9
- U1 pad 14: Net-(U1-Pad14) -> Switch8
- U1 pad 15: col5 -> Switch7
- U1 pad 16: col4 -> Switch6
- U1 pad 17: col3 -> Switch2
- U1 pad 18: col2 -> Switch3
- U1 pad 19: col1 -> Switch4
- U1 pad 20: col0 -> Switch5
- U1 pad 23: GND -> gnd
- U1 pad 24: Net-(U1-Pad24) -> raw
- U1 pad 3: GND -> gnd
- U1 pad 4: GND -> gnd
- U1 pad 5: SDA -> Switch11
- U1 pad 6: SCL -> Switch12
- U1 pad 7: row0 -> Switch13
- U1 pad 8: row1 -> Switch14
- U1 pad 9: row2 -> Switch15
Routing:
- net row0_r: track 163.2 -> 0.00 mm
- net row1_r: track 143.1 -> 0.00 mm
- net row2_r: track 132.5 -> 0.00 mm
- net Switch1: track 0.00 -> 131.8 mm, vias 0 -> 2
- net col5_r: track 131.0 -> 0.00 mm
- net Switch5: track 0.00 -> 122.3 mm, vias 0 -> 1
- net Switch2: track 0.00 -> 116.0 mm, vias 0 -> 1
- net Switch10: track 0.00 -> 114.6 mm, vias 0 -> 3
- net col4_r: track 114.5 -> 0.00 mm
- net Switch6: track 0.00 -> 109.2 mm, vias 0 -> 1
- net Switch4: track 0.00 -> 102.1 mm, vias 0 -> 1
- net Switch3: track 0.00 -> 100.9 mm, vias 0 -> 1
- net col3_r: track 97.9 -> 0.00 mm
- net Switch7: track 0.00 -> 90.6 mm, vias 0 -> 1
- net Switch15: track 0.00 -> 84.2 mm, vias 0 -> 2
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- added copper zone on B.Cu, net gnd
- added copper zone on F.Cu, net gnd
Other:
- board size 208.8 x 20 mm -> 89 x 71.2 mm
- rule pad_to_mask_clearance: 0.2 -> 0
- board text added: "B+"
- board text added: "B-"
- board text added: "Card34 by justalittleBIT"
- board text added: "Face down"
- board text added: "POWER SW"
